File: AmdekDaughterBoard/AmdekDaughterBoard.kicad_pcb (KiCad board)
At the start: 2 copper layers, 38.1 x 87.2 mm, 8 parts, among them J1 PINS 9-16, J2 PINS 1-8, U1 74LS257, U2 74LS257, U3 74LS161, U4 74LS161, U5 74LS161, U6 74LS161

Commit message: Add cable details, fab packages, instructions
Other:
- board text added: "1"
- board text added: "1/9"
- board text added: "8/16"
- board text added: "AmdekDVM"
