File: AmdekDaughterBoard/AmdekDaughterBoard.kicad_sch (KiCad schematic)
At the start: 8 parts, among them J1 PINS 9-16, J2 PINS 1-8, U1 74LS257, U2 74LS257, U3 74LS161, U4 74LS161, U5 74LS161, U6 74LS161

Commit message: Add cable details, fab packages, instructions
Changed lines of the file:
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@@
 	(text "B7"
 		(exclude_from_sim no)
-		(at 154.178 97.536 0)
+		(at 154.178 98.552 0)
 		(effects
 			(font
