File: AmdekDVM.kicad_sch (KiCad schematic)
At the start: 59 parts, among them J1 TO_DAUGHTERBOARD, J2 VIDEO, J3 APPLE II, U1 74LS123, U10 74LS04, U11 74LS74, U12 74LS04, U13 74LS10, U14 74LS10, U15 74LS10, U16 74LS08, U17 74LS11, U18 74LS08, U19 74LS04, U2 74LS175, U20 74LS51, U21 74LS95, U22 74LS164, U23 74LS95, U24 74LS00, U25 74LS54N, U26 74LS21, U27 74LS21, U28 74LS95, U29 74LS54N, U3 74LS157, U30 74LS54N, U31 74LS04, U32 74LS259, U33 74LS02, U34 74LS51, U35 74LS30, U36 74LS04, U37 74LS08, U38 74LS30, U4 74LS175, U5 SPARE, U6 74LS95, U7 74LS95, U8 74LS95, U9 74LS164

Commit message: Add daughterboards
Connections:
- net Net1 renamed H3
- net Net11 renamed H4
- net Net12 renamed H5
- net Net13 renamed VC
- net Net14 renamed V1
- net Net15 renamed V2
- net Net16 renamed V3
- net Net17 renamed V4
- net Net18 renamed D7
- net Net19 renamed D6
- net Net20 renamed D5
- net Net21 renamed D4
- net Net22 renamed D3
- net Net23 renamed D2
- net Net24 renamed D1
- net Net25 renamed D0
- net Net26 renamed ~{V1}
- net Net55 renamed WHT_D
- net Net56 renamed WHT
- net Net57 renamed VIO_GRN
- net Net58 renamed BLU_ORG
- net Net66 renamed ~{WHT}
- net Net67 renamed ~{BLU}
Other:
- note added: "1110x"
- note added: "grn#"
- note added: "red#"
- note added: "yel#"

Commit message: Add cable details, fab packages, instructions
Parts:
- added C14, C15, C16, C17, C18, C19, C20, C21, C22, C23: DNI, Capacitor_THT:C_Disc_D4.3mm_W1.9mm_P5.00mm, symbol Device:C_Small
Connections:
- net GND: now also C14.2, C15.2, C16.2, C17.2, C18.2, C19.2, C20.2, C21.2, C22.2, C23.2
- net VCC: now also C14.1, C15.1, C16.1, C17.1, C18.1, C19.1, C20.1, C21.1, C22.1, C23.1
Other:
- moved on the sheet: C10, C11, C12, C13, C3, C4, C5, C6, C7, C8, C9, R3

Commit message: Correct video pinout
Connections:
- net B_OUT: now also J2.3 (Pin_3), U33.1; no longer J2.2 (Pin_2), U33.10
- net G_OUT: now also J2.2 (Pin_2), U33.10; no longer J2.3 (Pin_3), U33.1
Changed lines of the file:
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@@
 	)
 	(label "G_OUT"
-		(at 662.94 505.46 0)
+		(at 662.94 530.86 0)
 		(effects
 			(font
@@
 	)
 	(label "B_OUT"
-		(at 662.94 530.86 0)
+		(at 662.94 505.46 0)
 		(effects
 			(font
@@
 	)
 	(label "G_OUT"
-		(at 709.93 501.65 180)
-		(effects
-			(font
-				(size 1.27 1.27)
-			)
-			(justify right bottom)
+		(at 722.63 499.11 0)
+		(effects
+			(font
+				(size 1.27 1.27)
+			)
+			(justify left bottom)
 		)
 	)
@@
 	)
 	(label "B_OUT"
-		(at 722.63 499.11 0)
-		(effects
-			(font
-				(size 1.27 1.27)
-			)
-			(justify left bottom)
-		)
-	)
+		(at 709.93 501.65 180)
+		(effects
+			(font
+				(size 1.27 1.27)
+			)
+			(justify right bottom)
+		)
+	)
